File: PSU/Xbox-PMS.kicad_pcb (KiCad board)
At the start: 4 copper layers, 121.2 x 34.2 mm, 150 parts, among them IC1 SIC437BED-T1-GE3, IC2 SIC437BED-T1-GE3, IC3 SIC437BED-T1-GE3, IC4 SIC437BED-T1-GE3, IC5 SIC437BED-T1-GE3, SW1 SW_Push, U1 MAX16054, U2 TPS61235PRWLT

Commit message: Delete HDMI Flipper Design Add HDMI Flex Add USB C/Power and volume button PCB Add Housing CAD Update IDE Flex Update S Controller PCBs Update LPC Flex Update USB Flex
Other:
- copper layers 4 -> 13
